File: AttenuverterFaceplate/AttenuverterFaceplate.kicad_pcb (KiCad board)
At the start: 2 copper layers, 30 x 128.5 mm, 17 parts

Commit message: Faceplate: squeezed wordmark footer, Orbitron text
Replaces the lower-left S-mark with the new 2mm-squeezed full wordmark
(_NTSFootprints:SchentronicsLogoSqueeze2mm), centered in the gap right
of the bottom screw hole (0.80mm margin each side). Adds ST-03, vertical,
centered in the left gap, anchored to the wordmark's bottom. Header and
part number switched from KiCad's italic stroke font to upright Orbitron.

Note: this file carries other pending local changes from before this
edit (titleblock/zone data), not just the faceplate update above.
Parts:
- removed the G*** at (130.2, 146.5)
- removed the REF** at (137.7, 151.2)
- removed the REF** at (137.7, 28.8)
- added G***: LOGO, _NTSFootprints:SchentronicsLogoSqueeze2mm, F.Cu at (135.2, 151.2)
Other:
- net class Default removed
- board text added: "ST-03"
