File: Attenuverter/Attenuverter.kicad_pcb (KiCad board)
At the start: 2 copper layers, 30 x 100 mm, 66 parts, among them J1 AudioJack2_SwitchT, J2 AudioJack2_SwitchT, J3 AudioJack2_SwitchT, J4 AudioJack2_SwitchT, J5 AudioJack2_SwitchT, J6 AudioJack2_SwitchT, J7 Conn_02x05_Odd_Even, J8 AudioJack2_SwitchT, J9 AudioJack2_SwitchT, U1 TL084, U2 LM4040DBZ-5

Commit message: PCB: align jacks to faceplate, nudge reference designators, add logo
- Move J1–J6, J8, J9 0.32 mm in X so the jack centers match the faceplate holes
  (faceplate centered on the board outline)
- Align reference designators to their neighbours (under 1 mm moves)
- Add the Schenktronics logo to the board
- Reroute the traces around the moved jacks
Parts:
- added G***: LOGO, _NTSFootprints:SchentronicsLogoSmed, B.Cu at (104.0, 53.6)
- moved J1 0.32 mm to (117.3, 55.0)
- moved J2 0.32 mm to (117.3, 67.0)
- moved J3 0.32 mm to (117.3, 81.0)
- moved J4 0.32 mm to (117.3, 93.0)
- moved J5 0.32 mm to (117.3, 107.0)
- moved J6 0.32 mm to (117.3, 119.0)
- moved J8 0.32 mm to (117.3, 133.0)
- moved J9 0.32 mm to (117.3, 145.0)

Commit message: Switch U1 to TL074, regenerate gerbers, and source U1/U2 from TI
- Change U1 from TL084 to TL074 in the schematic and PCB (same pinout)
- Source U1 (TL074CDR) and U2 (LM4040DBZ-5) from TI only, per the critical-IC rule
- Regenerate gerbers and drill files from the current board
Parts:
- U1: value TL084 -> TL074
Changed lines of the file:
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@@
 			)
 		)
-		(property "Value" "TL084"
+		(property "Value" "TL074"
 			(at 0 -5.28 90)
 			(layer "B.Fab")

Commit message: Add bottom-side fiducials and regenerate gerbers
- Add three 1 mm fiducials (2 mm mask opening) on the bottom side, clear of the jacks
- Move the logo off the fiducial area
- Regenerate gerbers, drill files and the zip, including the SMD pick-and-place file
Parts:
- added FID1: , Fiducial:Fiducial_1mm_Mask2mm, B.Cu at (103.0, 53.0)
- added FID2: , Fiducial:Fiducial_1mm_Mask2mm, B.Cu at (103.0, 133.0)
- added FID3: , Fiducial:Fiducial_1mm_Mask2mm, B.Cu at (113.0, 147.0)
- moved G*** 3.20 mm to (107.2, 53.6)
Changed lines of the file:
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@@
 		)
 	)
+	(footprint "Fiducial:Fiducial_1mm_Mask2mm"
+		(layer "B.Cu")
+		(at 113 147)
+		(descr "Fiducial, circular marking, 1mm bare copper, 2mm soldermask opening (Level A)")
+		(tags "fiducial")
+		(property "Reference" "FID3"
+			(at 0 -1.95 0)
+			(layer "B.SilkS")
+			(hide yes)
+			(effects
+				(font
+					(size 1 1)
+					(thickness 0.15)
+				)
+			)
+		)
+		(property "Value" ""
+			(at 0 0 0)
+			(layer "F.Fab")
+			(effects
+				(font
+					(size 1.27 1.27)
+				)
+			)
+		)
+		(property "Datasheet" ""
+			(at 0 0 0)
+			(layer "F.Fab")
+			(hide yes)
+			(effects
+				(font
+					(size 1.27 1.27)
+				)
+			)
+		)
+		(property "Description" ""
+			(at 0 0 0)
+			(layer "F.Fab")
+			(hide yes)
+			(effects
+				(font
+					(size 1.27 1.27)
+				)
+			)
+		)
+		(attr smd exclude_from_bom)
+		(duplicate_pad_numbers_are_jumpers no)
+		(fp_circle
+			(center 0 0)
+			(end 1.25 0)
+			(stroke
+				(width 0.05)
+				(type solid)
+			)
+			(fill no)
+			(layer "B.CrtYd")
+		)
+		(fp_circle
+			(center 0 0)
+			(end 1 0)
+			(stroke
+				(width 0.1)
+				(type solid)
+			)
+			(fill no)
+			(layer "B.Fab")
+		)
+		(pad "" smd circle
+			(at 0 0)
+			(size 1 1)
+			(layers "B.Cu" "B.Mask")
+			(solder_mask_margin 0.5)
+			(clearance 0.6)
+		)
+		(embedded_fonts no)
+	)
 	(footprint "Diode_SMD:D_SOD-323"
 		(layer "B.Cu")
@@
 		)
 	)
+	(footprint "Fiducial:Fiducial_1mm_Mask2mm"
+		(layer "B.Cu")
+		(at 103 133)
+		(descr "Fiducial, circular marking, 1mm bare copper, 2mm soldermask opening (Level A)")
+		(tags "fiducial")
+		(property "Reference" "FID2"
+			(at 0 -1.95 0)
+			(layer "B.SilkS")
+			(hide yes)
+			(effects
+				(font
+					(size 1 1)
+					(thickness 0.15)
+				)
+			)
+		)
+		(property "Value" ""
+			(at 0 0 0)
+			(layer "F.Fab")
+			(effects
+				(font
+					(size 1.27 1.27)
+				)
+			)
+		)
+		(property "Datasheet" ""
+			(at 0 0 0)
+			(layer "F.Fab")
+			(hide yes)
+			(effects
+				(font
+					(size 1.27 1.27)
+				)
+			)
+		)
+		(property "Description" ""
+			(at 0 0 0)
+			(layer "F.Fab")
+			(hide yes)
+			(effects
+				(font
+					(size 1.27 1.27)
+				)
+			)
+		)
+		(attr smd exclude_from_bom)
+		(duplicate_pad_numbers_are_jumpers no)
+		(fp_circle
+			(center 0 0)
+			(end 1.25 0)
+			(stroke
+				(width 0.05)
+				(type solid)
+			)
+			(fill no)
+			(layer "B.CrtYd")
+		)
+		(fp_circle
+			(center 0 0)
+			(end 1 0)
+			(stroke
+				(width 0.1)
+				(type solid)
+			)
+			(fill no)
+			(layer "B.Fab")
+		)
+		(pad "" smd circle
+			(at 0 0)
+			(size 1 1)
+			(layers "B.Cu" "B.Mask")
+			(solder_mask_margin 0.5)
+			(clearance 0.6)
+		)
+		(embedded_fonts no)
+	)
+	(footprint "Fiducial:Fiducial_1mm_Mask2mm"
+		(layer "B.Cu")
+		(at 103 53)
+		(descr "Fiducial, circular marking, 1mm bare copper, 2mm soldermask opening (Level A)")
+		(tags "fiducial")
+		(property "Reference" "FID1"
+			(at 0 -1.95 0)
+			(layer "B.SilkS")
+			(hide yes)
+			(effects
+				(font
+					(size 1 1)
+					(thickness 0.15)
+				)
+			)
+		)
+		(property "Value" ""
+			(at 0 0 0)
+			(layer "F.Fab")
+			(effects
+				(font
+					(size 1.27 1.27)
+				)
+			)
+		)
+		(property "Datasheet" ""
+			(at 0 0 0)
+			(layer "F.Fab")
+			(hide yes)
+			(effects
+				(font
+					(size 1.27 1.27)
+				)
+			)
+		)
+		(property "Description" ""
+			(at 0 0 0)
+			(layer "F.Fab")
+			(hide yes)
+			(effects
+				(font
+					(size 1.27 1.27)
+				)
+			)
+		)
+		(attr smd exclude_from_bom)
+		(duplicate_pad_numbers_are_jumpers no)
+		(fp_circle
+			(center 0 0)
+			(end 1.25 0)
+			(stroke
+				(width 0.05)
+				(type solid)
+			)
+			(fill no)
+			(layer "B.CrtYd")
+		)
+		(fp_circle
+			(center 0 0)
+			(end 1 0)
+			(stroke
+				(width 0.1)
+				(type solid)
+			)
+			(fill no)
+			(layer "B.Fab")
+		)
+		(pad "" smd circle
+			(at 0 0)
+			(size 1 1)
+			(layers "B.Cu" "B.Mask")
+			(solder_mask_margin 0.5)
+			(clearance 0.6)
+		)
+		(embedded_fonts no)
+	)
 	(footprint "Diode_SMD:D_SOD-323"
 		(layer "B.Cu")
@@
 	(footprint "_NTSFootprints:SchentronicsLogoSmed"
 		(layer "B.Cu")
-		(at 104 53.6 180)
+		(at 107.2 53.6 180)
 		(property "Reference" "G***"
 			(at 0 0 0)

Commit message: Use LM4040DIM3X-5.0/NOPB for U2
- Set the U2 value on the schematic and PCB to LM4040DIM3X-5.0/NOPB
- Update the BOM to match, and regenerate gerbers, drill files, zip and the SMD CPL
Parts:
- U2: value LM4040DBZ-5 -> LM4040DIM3X-5.0/NOPB
Changed lines of the file:
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@@
 			)
 		)
-		(property "Value" "LM4040DBZ-5"
+		(property "Value" "LM4040DIM3X-5.0/NOPB"
 			(at 0 -2.4 180)
 			(layer "B.Fab")

Commit message: Update PCB version label to v1.1
Other:
- board text added: "Attenuverter v1.1"
- board text removed: "Attenuverter v1.0"
Changed lines of the file:
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@@
 		(layer "Edge.Cuts")
 	)
-	(gr_text "Attenuverter\nv1.0"
+	(gr_text "Attenuverter\nv1.1"
 		(at 113.5 128.25 0)
 		(layer "B.SilkS")
