File: Attenuverter/Attenuverter.kicad_pcb (KiCad board)
At the start: 2 copper layers, 30 x 100 mm, 70 parts, among them J1 AudioJack2_SwitchT, J2 AudioJack2_SwitchT, J3 AudioJack2_SwitchT, J4 AudioJack2_SwitchT, J5 AudioJack2_SwitchT, J6 AudioJack2_SwitchT, J7 Conn_02x05_Odd_Even, J8 AudioJack2_SwitchT, J9 AudioJack2_SwitchT, U1 TL074, U2 LM4040DIM3X-5.0/NOPB

Commit message: Main PCB: harmonize branding text with the Multiple's pattern
Reformatted "Attenuverter\nv1.1" to "ST-03 v1.1\nAttenuverter" (code +
version first, name second), matching the Multiple's layout convention.
Logo stays as the medium S-mark, already in a clear spot.

Tried adding the CC BY-NC-SA roundels + text too, matching the Multiple,
but this board is far more densely routed (active circuit vs. the
Multiple's passive jacks-only layout) -- verified via kicad-cli renders
that every candidate spot collided with real pads or traces, so left
them off rather than force an overlap. Space, not a fixed rule, is
what decided this per board.
Other:
- board text added: "ST-03 v1.1 Attenuverter"
- board text removed: "Attenuverter v1.1"
Changed lines of the file:
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@@
 		(layer "Edge.Cuts")
 	)
-	(gr_text "Attenuverter\nv1.1"
+	(gr_text "ST-03 v1.1\nAttenuverter"
 		(at 113.5 128.25 0)
 		(layer "B.SilkS")
