File: Attenuverter/Attenuverter.kicad_sch (KiCad schematic)
At the start: 66 parts, among them J1 AudioJack2_SwitchT, J2 AudioJack2_SwitchT, J3 AudioJack2_SwitchT, J4 AudioJack2_SwitchT, J5 AudioJack2_SwitchT, J6 AudioJack2_SwitchT, J7 Conn_02x05_Odd_Even, J8 AudioJack2_SwitchT, J9 AudioJack2_SwitchT, U1 TL084, U2 LM4040DBZ-5

Commit message: Switch U1 to TL074, regenerate gerbers, and source U1/U2 from TI
- Change U1 from TL084 to TL074 in the schematic and PCB (same pinout)
- Source U1 (TL074CDR) and U2 (LM4040DBZ-5) from TI only, per the critical-IC rule
- Regenerate gerbers and drill files from the current board
Parts:
- U1: value TL084 -> TL074; symbol Amplifier_Operational:TL084 -> Amplifier_Operational:TL074
Changed lines of the file:
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@@
 	)
 	(symbol
-		(lib_id "Amplifier_Operational:TL084")
+		(lib_id "Amplifier_Operational:TL074")
 		(at 218.44 101.6 0)
 		(unit 5)
@@
 			)
 		)
-		(property "Value" "TL084"
+		(property "Value" "TL074"
 			(at 217.3732 102.743 0)
 			(show_name no)
@@
 			)
 		)
-		(property "Datasheet" "http://www.ti.com/lit/ds/symlink/tl081.pdf"
+		(property "Datasheet" "http://www.ti.com/lit/ds/symlink/tl071.pdf"
 			(at 219.71 96.52 0)
 			(hide yes)
@@
 	)
 	(symbol
-		(lib_id "Amplifier_Operational:TL084")
+		(lib_id "Amplifier_Operational:TL074")
 		(at 85.09 41.91 0)
 		(mirror x)
@@
 			)
 		)
-		(property "Value" "TL084"
+		(property "Value" "TL074"
 			(at 87.63 36.83 0)
 			(show_name no)
@@
 			)
 		)
-		(property "Datasheet" "http://www.ti.com/lit/ds/symlink/tl081.pdf"
+		(property "Datasheet" "http://www.ti.com/lit/ds/symlink/tl071.pdf"
 			(at 86.36 46.99 0)
 			(hide yes)
@@
 	)
 	(symbol
-		(lib_id "Amplifier_Operational:TL084")
+		(lib_id "Amplifier_Operational:TL074")
 		(at 85.09 80.01 0)
 		(mirror x)
@@
 			)
 		)
-		(property "Value" "TL084"
+		(property "Value" "TL074"
 			(at 87.63 74.93 0)
 			(show_name no)
@@
 			)
 		)
-		(property "Datasheet" "http://www.ti.com/lit/ds/symlink/tl081.pdf"
+		(property "Datasheet" "http://www.ti.com/lit/ds/symlink/tl071.pdf"
 			(at 86.36 85.09 0)
 			(hide yes)
@@
 	)
 	(symbol
-		(lib_id "Amplifier_Operational:TL084")
+		(lib_id "Amplifier_Operational:TL074")
 		(at 85.09 118.11 0)
 		(mirror x)
@@
 			)
 		)
-		(property "Value" "TL084"
+		(property "Value" "TL074"
 			(at 87.63 113.03 0)
 			(show_name no)
@@
 			)
 		)
-		(property "Datasheet" "http://www.ti.com/lit/ds/symlink/tl081.pdf"
+		(property "Datasheet" "http://www.ti.com/lit/ds/symlink/tl071.pdf"
 			(at 86.36 123.19 0)
 			(hide yes)
@@
 	)
 	(symbol
-		(lib_id "Amplifier_Operational:TL084")
+		(lib_id "Amplifier_Operational:TL074")
 		(at 85.09 156.21 0)
 		(mirror x)
@@
 			)
 		)
-		(property "Value" "TL084"
+		(property "Value" "TL074"
 			(at 87.63 151.13 0)
 			(show_name no)
@@
 			)
 		)
-		(property "Datasheet" "http://www.ti.com/lit/ds/symlink/tl081.pdf"
+		(property "Datasheet" "http://www.ti.com/lit/ds/symlink/tl071.pdf"
 			(at 86.36 161.29 0)
 			(hide yes)

Commit message: Use LM4040DIM3X-5.0/NOPB for U2
- Set the U2 value on the schematic and PCB to LM4040DIM3X-5.0/NOPB
- Update the BOM to match, and regenerate gerbers, drill files, zip and the SMD CPL
Parts:
- U2: value LM4040DBZ-5 -> LM4040DIM3X-5.0/NOPB
Changed lines of the file:
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@@
 			)
 		)
-		(property "Value" "LM4040DBZ-5"
+		(property "Value" "LM4040DIM3X-5.0/NOPB"
 			(at 224.79 107.95 90)
 			(show_name no)

Commit message: Label input clamp diodes as 1N4148WS-7-F
Parts:
- D10, D11, D3, D4, D5, D6, D7, D8, D9: value D -> 1N4148WS-7-F
Changed lines of the file:
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@@
 			)
 		)
-		(property "Value" "D"
+		(property "Value" "1N4148WS-7-F"
 			(at 47.7266 151.003 90)
 			(hide yes)
@@
 			)
 		)
-		(property "Value" "D"
+		(property "Value" "1N4148WS-7-F"
 			(at 47.7266 74.803 90)
 			(hide yes)
@@
 			)
 		)
-		(property "Value" "D"
+		(property "Value" "1N4148WS-7-F"
 			(at 47.7266 82.423 90)
 			(hide yes)
@@
 			)
 		)
-		(property "Value" "D"
+		(property "Value" "1N4148WS-7-F"
 			(at 47.7266 120.523 90)
 			(hide yes)
@@
 			)
 		)
-		(property "Value" "D"
+		(property "Value" "1N4148WS-7-F"
 			(at 47.7266 36.703 90)
 			(hide yes)
@@
 			)
 		)
-		(property "Value" "D"
+		(property "Value" "1N4148WS-7-F"
 			(at 47.7266 158.623 90)
 			(hide yes)
@@
 			)
 		)
-		(property "Value" "D"
+		(property "Value" "1N4148WS-7-F"
 			(at 264.8966 107.823 90)
 			(hide yes)
@@
 			)
 		)
-		(property "Value" "D"
+		(property "Value" "1N4148WS-7-F"
 			(at 47.7266 44.323 90)
 			(hide yes)
@@
 			)
 		)
-		(property "Value" "D"
+		(property "Value" "1N4148WS-7-F"
 			(at 47.7266 112.903 90)
 			(hide yes)

Commit message: Title blocks: logo worksheet, consistent company/rev across PCB and schematic
Repoint page_layout_descr_file (both pcbnew and schematic) from the old
Windows path to the real one on this machine, so the Schenktronics
worksheet -- and its embedded logo -- actually loads.

Fill out/correct title blocks: company standardized to "Schenktronics"
(was "Nathan Schenk"), and PCB rev brought up to 1.1 to match both the
real "v1.1" silkscreen text and the schematic's already-correct 1.1 --
the PCB title block had been stuck at the old 1.0. Faceplate matched to
the same 1.1 for consistency within the product.
Other:
- company: Nathan Schenk -> Schenktronics
Changed lines of the file:
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@@
 		(date "2026-10-03")
 		(rev "1.1")
-		(company "Nathan Schenk")
+		(company "Schenktronics")
 	)
 	(junction
