File: hardware/attenuverter/Attenuverter.kicad_pcb (KiCad board)
At the start: 2 copper layers, 30 x 100 mm, 70 parts, among them J1 AudioJack2_SwitchT, J2 AudioJack2_SwitchT, J3 AudioJack2_SwitchT, J4 AudioJack2_SwitchT, J5 AudioJack2_SwitchT, J6 AudioJack2_SwitchT, J7 Conn_02x05_Odd_Even, J8 AudioJack2_SwitchT, J9 AudioJack2_SwitchT, U1 TL074, U2 LM4040DIM3X-5.0/NOPB

Commit message: Update footprints
Parts:
- D10, D11, D3, D4, D5, D6, D7, D8, D9: value D -> 1N4148WS-7-F
- U2: value LM4040DIM3X-5.0/NOPB -> LM4040D50IDBZR
