File: hardware/attenuverter/Attenuverter.kicad_sch (KiCad schematic)
At the start: 66 parts, among them J1 AudioJack2_SwitchT, J2 AudioJack2_SwitchT, J3 AudioJack2_SwitchT, J4 AudioJack2_SwitchT, J5 AudioJack2_SwitchT, J6 AudioJack2_SwitchT, J7 Conn_02x05_Odd_Even, J8 AudioJack2_SwitchT, J9 AudioJack2_SwitchT, U1 TL074, U2 LM4040DIM3X-5.0/NOPB

Commit message: Switch to a non-detent pot; fix an obsolete LM4040 part number
New BOM: Bourns PTV09A-4020F-B104 (bushingless, no center detent),
replacing PTV09A-4225F-B104. Same mounting style and KiCad footprint as
before (both are the PTV09 family's bushingless rear-mount variant,
differing only in shaft length and detent option per Bourns' ordering
code), so no footprint change is needed — only the BOM, the docs that
described the detent, and the panel/patch drawing scripts' comments.
The knob (Davies 1221-J) is unchanged.

Also fixes U2's part number: the old LM4040DIM3X-5.0/NOPB (TI's legacy
M3X-suffix ordering format) showed up Obsolete with no price at Mouser.
TI's current datasheet confirms the LM4040 family itself is still
Active — TI just moved to a shorter orderable-number format between
the January 2015 and October 2017 datasheet revisions.
LM4040D50IDBZR is the current listing for the same grade/voltage/
package, live at Mouser.
Parts:
- U2: value LM4040DIM3X-5.0/NOPB -> LM4040D50IDBZR
Changed lines of the file:
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@@
 			)
 		)
-		(property "Value" "LM4040DIM3X-5.0/NOPB"
+		(property "Value" "LM4040D50IDBZR"
 			(at 224.79 107.95 90)
 			(show_name no)

Commit message: Update footprints
Parts:
- C1, C2, C3, C4, C5, C6, C7, C8, C9: footprint Capacitors_SMD:C_0805_HandSoldering -> Capacitor_SMD:C_0805_2012Metric
- D1, D2: footprint Diodes_SMD:D_SMA_Handsoldering -> Diode_SMD:D_SMA
- F1, F2: footprint Fuse_Holders_and_Fuses:Fuse_SMD1206_HandSoldering -> Fuse:Fuse_1206_3216Metric
- R1, R10, R11, R12, R13, R14, R15, R16, R17, R18, R19, R2, R20, R21, R22, R23, R24, R25, R26, R27, R28, R29, R3, R4, R5, R6, R7, R8, R9: footprint Resistors_SMD:R_0805_HandSoldering -> Resistor_SMD:R_0805_2012Metric
- U1: footprint Housings_SOIC:SOIC-14_3.9x8.7mm_Pitch1.27mm -> Package_SO:SOIC-14_3.9x8.7mm_P1.27mm
- U2: footprint TO_SOT_Packages_SMD:SOT-23 -> Package_TO_SOT_SMD:SOT-23
Changed lines of the file:
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@@
 			)
 		)
-		(property "Footprint" "Housings_SOIC:SOIC-14_3.9x8.7mm_Pitch1.27mm"
+		(property "Footprint" "Package_SO:SOIC-14_3.9x8.7mm_P1.27mm"
 			(at 217.17 99.06 0)
 			(hide yes)
@@
 			)
 		)
-		(property "Footprint" "Housings_SOIC:SOIC-14_3.9x8.7mm_Pitch1.27mm"
+		(property "Footprint" "Package_SO:SOIC-14_3.9x8.7mm_P1.27mm"
 			(at 83.82 44.45 0)
 			(hide yes)
@@
 			)
 		)
-		(property "Footprint" "Resistors_SMD:R_0805_HandSoldering"
+		(property "Footprint" "Resistor_SMD:R_0805_2012Metric"
 			(at 85.09 32.512 90)
 			(hide yes)
@@
 			)
 		)
-		(property "Footprint" "Resistors_SMD:R_0805_HandSoldering"
+		(property "Footprint" "Resistor_SMD:R_0805_2012Metric"
 			(at 71.12 37.592 90)
 			(hide yes)
@@
 			)
 		)
-		(property "Footprint" "Resistors_SMD:R_0805_HandSoldering"
+		(property "Footprint" "Resistor_SMD:R_0805_2012Metric"
 			(at 65.278 43.18 90)
 			(hide yes)
@@
 			)
 		)
-		(property "Footprint" "Resistors_SMD:R_0805_HandSoldering"
+		(property "Footprint" "Resistor_SMD:R_0805_2012Metric"
 			(at 65.278 50.8 90)
 			(hide yes)
@@
 			)
 		)
-		(property "Footprint" "Resistors_SMD:R_0805_HandSoldering"
+		(property "Footprint" "Resistor_SMD:R_0805_2012Metric"
 			(at 99.06 40.132 90)
 			(hide yes)
@@
 			)
 		)
-		(property "Footprint" "Capacitors_SMD:C_0805_HandSoldering"
+		(property "Footprint" "Capacitor_SMD:C_0805_2012Metric"
 			(at 81.28 26.3652 0)
 			(hide yes)
@@
 			)
 		)
-		(property "Footprint" "TO_SOT_Packages_SMD:SOT-23"
+		(property "Footprint" "Package_TO_SOT_SMD:SOT-23"
 			(at 246.38 106.68 0)
 			(hide yes)
@@
 			)
 		)
-		(property "Footprint" "Resistors_SMD:R_0805_HandSoldering"
+		(property "Footprint" "Resistor_SMD:R_0805_2012Metric"
 			(at 243.078 96.52 90)
 			(hide yes)
@@
 			)
 		)
-		(property "Footprint" "Capacitors_SMD:C_0805_HandSoldering"
+		(property "Footprint" "Capacitor_SMD:C_0805_2012Metric"
 			(at 252.4252 110.49 0)
 			(hide yes)
@@
 			)
 		)
-		(property "Footprint" "Housings_SOIC:SOIC-14_3.9x8.7mm_Pitch1.27mm"
+		(property "Footprint" "Package_SO:SOIC-14_3.9x8.7mm_P1.27mm"
 			(at 83.82 82.55 0)
 			(hide yes)
@@
 			)
 		)
-		(property "Footprint" "Resistors_SMD:R_0805_HandSoldering"
+		(property "Footprint" "Resistor_SMD:R_0805_2012Metric"
 			(at 85.09 70.612 90)
 			(hide yes)
@@
 			)
 		)
-		(property "Footprint" "Resistors_SMD:R_0805_HandSoldering"
+		(property "Footprint" "Resistor_SMD:R_0805_2012Metric"
 			(at 71.12 75.692 90)
 			(hide yes)
@@
 			)
 		)
-		(property "Footprint" "Resistors_SMD:R_0805_HandSoldering"
+		(property "Footprint" "Resistor_SMD:R_0805_2012Metric"
 			(at 65.278 81.28 90)
 			(hide yes)
@@
 			)
 		)
-		(property "Footprint" "Resistors_SMD:R_0805_HandSoldering"
+		(property "Footprint" "Resistor_SMD:R_0805_2012Metric"
 			(at 65.278 88.9 90)
 			(hide yes)
@@
 			)
 		)
-		(property "Footprint" "Resistors_SMD:R_0805_HandSoldering"
+		(property "Footprint" "Resistor_SMD:R_0805_2012Metric"
 			(at 99.06 78.232 90)
 			(hide yes)
@@
 			)
 		)
-		(property "Footprint" "Capacitors_SMD:C_0805_HandSoldering"
+		(property "Footprint" "Capacitor_SMD:C_0805_2012Metric"
 			(at 81.28 64.4652 0)
 			(hide yes)
@@
 			)
 		)
-		(property "Footprint" "Housings_SOIC:SOIC-14_3.9x8.7mm_Pitch1.27mm"
+		(property "Footprint" "Package_SO:SOIC-14_3.9x8.7mm_P1.27mm"
 			(at 83.82 120.65 0)
 			(hide yes)
@@
 			)
 		)
-		(property "Footprint" "Resistors_SMD:R_0805_HandSoldering"
+		(property "Footprint" "Resistor_SMD:R_0805_2012Metric"
 			(at 85.09 108.712 90)
 			(hide yes)
@@
 			)
 		)
-		(property "Footprint" "Resistors_SMD:R_0805_HandSoldering"
+		(property "Footprint" "Resistor_SMD:R_0805_2012Metric"
 			(at 71.12 113.792 90)
 			(hide yes)
@@
 			)
 		)
-		(property "Footprint" "Resistors_SMD:R_0805_HandSoldering"
+		(property "Footprint" "Resistor_SMD:R_0805_2012Metric"
 			(at 65.278 119.38 90)
 			(hide yes)
@@
 			)
 		)
-		(property "Footprint" "Resistors_SMD:R_0805_HandSoldering"
+		(property "Footprint" "Resistor_SMD:R_0805_2012Metric"
 			(at 65.278 127 90)
 			(hide yes)
@@
 			)
 		)
-		(property "Footprint" "Resistors_SMD:R_0805_HandSoldering"
+		(property "Footprint" "Resistor_SMD:R_0805_2012Metric"
 			(at 99.06 116.332 90)
 			(hide yes)
@@
 			)
 		)
-		(property "Footprint" "Capacitors_SMD:C_0805_HandSoldering"
+		(property "Footprint" "Capacitor_SMD:C_0805_2012Metric"
 			(at 81.28 102.5652 0)
 			(hide yes)
@@
 			)
 		)
-		(property "Footprint" "Housings_SOIC:SOIC-14_3.9x8.7mm_Pitch1.27mm"
+		(property "Footprint" "Package_SO:SOIC-14_3.9x8.7mm_P1.27mm"
 			(at 83.82 158.75 0)
 			(hide yes)
@@
 			)
 		)
-		(property "Footprint" "Resistors_SMD:R_0805_HandSoldering"
+		(property "Footprint" "Resistor_SMD:R_0805_2012Metric"
 			(at 85.09 146.812 90)
 			(hide yes)
@@
 			)
 		)
-		(property "Footprint" "Resistors_SMD:R_0805_HandSoldering"
+		(property "Footprint" "Resistor_SMD:R_0805_2012Metric"
 			(at 71.12 151.892 90)
 			(hide yes)
@@
 			)
 		)
-		(property "Footprint" "Resistors_SMD:R_0805_HandSoldering"
+		(property "Footprint" "Resistor_SMD:R_0805_2012Metric"
 			(at 65.278 157.48 90)
 			(hide yes)
@@
 			)
 		)
-		(property "Footprint" "Resistors_SMD:R_0805_HandSoldering"
+		(property "Footprint" "Resistor_SMD:R_0805_2012Metric"
 			(at 65.278 165.1 90)
 			(hide yes)
@@
 			)
 		)
-		(property "Footprint" "Resistors_SMD:R_0805_HandSoldering"
+		(property "Footprint" "Resistor_SMD:R_0805_2012Metric"
 			(at 99.06 154.432 90)
 			(hide yes)
@@
 			)
 		)
-		(property "Footprint" "Capacitors_SMD:C_0805_HandSoldering"
+		(property "Footprint" "Capacitor_SMD:C_0805_2012Metric"
 			(at 81.28 140.6652 0)
 			(hide yes)
@@
 			)
 		)
-		(property "Footprint" "Capacitors_SMD:C_0805_HandSoldering"
+		(property "Footprint" "Capacitor_SMD:C_0805_2012Metric"
 			(at 216.8652 138.43 0)
 			(hide yes)
@@
 			)
 		)
-		(property "Footprint" "Capacitors_SMD:C_0805_HandSoldering"
+		(property "Footprint" "Capacitor_SMD:C_0805_2012Metric"
 			(at 216.8652 148.59 0)
 			(hide yes)
@@
 			)
 		)
-		(property "Footprint" "Capacitors_SMD:C_0805_HandSoldering"
+		(property "Footprint" "Capacitor_SMD:C_0805_2012Metric"
 			(at 204.1652 138.43 0)
 			(hide yes)
@@
 			)
 		)
-		(property "Footprint" "Capacitors_SMD:C_0805_HandSoldering"
+		(property "Footprint" "Capacitor_SMD:C_0805_2012Metric"
 			(at 204.1652 148.59 0)
 			(hide yes)
@@
 			)
 		)
-		(property "Footprint" "Fuse_Holders_and_Fuses:Fuse_SMD1206_HandSoldering"
+		(property "Footprint" "Fuse:Fuse_1206_3216Metric"
 			(at 246.38 135.89 0)
 			(hide yes)
@@
 			)
 		)
-		(property "Footprint" "Diodes_SMD:D_SMA_Handsoldering"
+		(property "Footprint" "Diode_SMD:D_SMA"
 			(at 241.3 135.89 0)
 			(hide yes)
@@
 			)
 		)
-		(property "Footprint" "Fuse_Holders_and_Fuses:Fuse_SMD1206_HandSoldering"
+		(property "Footprint" "Fuse:Fuse_1206_3216Metric"
 			(at 246.38 146.05 0)
 			(hide yes)
@@
 			)
 		)
-		(property "Footprint" "Diodes_SMD:D_SMA_Handsoldering"
+		(property "Footprint" "Diode_SMD:D_SMA"
 			(at 241.3 143.51 0)
 			(hide yes)
@@
 			)
 		)
-		(property "Footprint" "Resistors_SMD:R_0805_HandSoldering"
+		(property "Footprint" "Resistor_SMD:R_0805_2012Metric"
 			(at 36.322 30.48 90)
 			(hide yes)
@@
 			)
 		)
-		(property "Footprint" "Resistors_SMD:R_0805_HandSoldering"
+		(property "Footprint" "Resistor_SMD:R_0805_2012Metric"
 			(at 36.322 144.78 90)
 			(hide yes)
@@
 			)
 		)
-		(property "Footprint" "Resistors_SMD:R_0805_HandSoldering"
+		(property "Footprint" "Resistor_SMD:R_0805_2012Metric"
 			(at 38.1 79.248 90)
 			(hide yes)
@@
 			)
 		)
-		(property "Footprint" "Resistors_SMD:R_0805_HandSoldering"
+		(property "Footprint" "Resistor_SMD:R_0805_2012Metric"
 			(at 38.1 155.448 90)
 			(hide yes)
@@
 			)
 		)
-		(property "Footprint" "Resistors_SMD:R_0805_HandSoldering"
+		(property "Footprint" "Resistor_SMD:R_0805_2012Metric"
 			(at 38.1 117.348 90)
 			(hide yes)
@@
 			)
 		)
-		(property "Footprint" "Resistors_SMD:R_0805_HandSoldering"
+		(property "Footprint" "Resistor_SMD:R_0805_2012Metric"
 			(at 36.322 106.68 90)
 			(hide yes)
@@
 			)
 		)
-		(property "Footprint" "Resistors_SMD:R_0805_HandSoldering"
+		(property "Footprint" "Resistor_SMD:R_0805_2012Metric"
 			(at 36.322 68.58 90)
 			(hide yes)
@@
 			)
 		)
-		(property "Footprint" "Resistors_SMD:R_0805_HandSoldering"
+		(property "Footprint" "Resistor_SMD:R_0805_2012Metric"
 			(at 38.1 41.148 90)
 			(hide yes)
